Commit message: added object types, and obj_env run_env controls individual joints

File: warp/envs/assets/Bottle/3558/mobility.urdf (robot description, URDF)
Before this commit: robot partnet_158634b1d7d010eeebe67d9b32c3ddf8, 4 links, 3 joints
Joints:
- joint joint_2: limit lower=-0.1080000000000001 upper=0 -> lower=-0.1080000000000001 upper=0 effort=100.0 velocity=1

File: warp/envs/assets/Dispenser/101417/mobility.urdf (robot description, URDF)
Before this commit: robot partnet_2a9b20d21e27ab0026cca18be86a1458, 5 links, 4 joints
Joints:
- joint joint_0: limit lower=0.0 upper=0.5215043804959058 -> lower=0.0 upper=0.5215043804959058 effort=100.0 velocity=1
- joint joint_3: limit lower=0 upper=0.12 -> lower=0 upper=0.12 effort=100.0 velocity=1

File: warp/envs/assets/Stapler/103271/mobility.urdf (robot description, URDF)
Before this commit: robot partnet_8c34afa29665356013b1d3e1528f0506-0, 4 links, 3 joints
Joints:
- joint joint_2: origin xyz=0 0 0 rpy=1.570796326794897 0 -1.570796326794897 -> xyz=0 0 0 rpy=1.570796326794897 1.57 -1.570796326794897
