Commit message: added grasp data and grasp tests

File: warp/envs/assets/USB/102052/mobility.urdf (robot description, URDF)
Before this commit: robot partnet_e1791a5d41be53db620b4d027d55e817-0, 3 links, 2 joints
Links:
- added link link_0_helper
- link link_1: geometry collision mesh filename=textured_objs/new-1.obj; collision mesh filename=textured_objs/new-3.obj
Joints:
- added joint joint_2: type prismatic, parent link_1, child link_0_helper, origin xyz=-0.002291089456653725 0 -0.014289999999999997, axis 0 1 0, limit lower=-0.06400000000000006 upper=0.2639999999999998 effort=100 velocity=1
- joint joint_0: axis 0 0 1 -> 0 1 0; limit lower=-0.3480000000000001 upper=-0.08 -> (none); origin xyz=0 0 0 -> xyz=0.0 0 0.0; parent link_1 -> link_0_helper; type prismatic -> continuous
