Commit message: fixed joints in stapler to remove middle joint artifacts

File: warp/envs/assets/Dispenser/101539/mobility.urdf (robot description, URDF)
Before this commit: robot partnet_a1c91a0d66c865b0c0ea4586d3cf4a4, 4 links, 3 joints
Joints:
- joint joint_0: limit (none) -> lower=-0.05 upper=0.2; type continuous -> prismatic

File: warp/envs/assets/Stapler/102990/mobility.urdf (robot description, URDF)
Before this commit: robot partnet_20c5096ea98cc955920de219c00d1c3b, 4 links, 3 joints
Joints:
- joint joint_0: origin xyz=0 0.0 0.0 -> xyz=0.0 0.0 0.0 rpy=-0.15 0. 0.

File: warp/envs/assets/Stapler/103271/mobility.urdf (robot description, URDF)
Before this commit: robot partnet_8c34afa29665356013b1d3e1528f0506-0, 4 links, 3 joints
Joints:
- joint joint_0: type revolute -> fixed

File: warp/envs/assets/Stapler/103792/mobility.urdf (robot description, URDF)
Before this commit: robot partnet_88ac7b2b3050f1f861f7b52424be58ab, 4 links, 3 joints
Joints:
- joint joint_0: type revolute -> fixed
