Commit message: updated object grasp loading to boolean flag in handenv, updates to partnet continuous joint

File: warp/envs/assets/pill_bottle/mobility.urdf (robot description, URDF)
Before this commit: robot partnet_fdc47f5f8dff184830eaaf40a8a562c1, 4 links, 3 joints
Joints:
- joint joint_0: origin xyz=0.0 0 0.0 -> xyz=0.0 0.0 0.0
